File: Domowy Sterownik GSM.sch (KiCad schematic (older format))
At the start: 98 parts

Commit message: 2
Parts:
- removed IC?: TLP281-4, SOP16, symbol TLP291-4
Changed lines of the file:
@@
 Sheet 1 1
 Title "Domowy Sterownik GSM"
-Date "16 mar 2015"
+Date "17 mar 2015"
 Rev ""
 Comp "Marcin Kowalski, Łukasz Tim, Adrian Wrotecki"
@@
 	1    0    0    -1
 $EndComp
-$Comp
-L TLP291-4 IC?
-U 1 1 55074DC5
-P 1850 6650
-F 0 "IC?" H 1662 6828 40  0000 C CNN
-F 1 "TLP281-4" H 1949 6466 40  0000 C CNN
-F 2 "SOP16" H 1686 6476 29  0000 C CNN
-F 3 "" H 1850 6650 60  0000 C CNN
-	1    1850 6650
-	1    0    0    -1
-$EndComp
